Commit message: Description updates for accuracy and fixing footprint

File: limo_description/urdf/limo_ackerman.xacro (robot description, xacro)
@@ -19,7 +19,7 @@
     <link name="base_footprint"/>
     <joint name="base_joint" type="fixed">
-    <parent link="base_footprint"/>
-    <child link="base_link"/>
-    <origin xyz="0.0 0.0 0.15" rpy="0 0 0"/>
+    <parent link="base_link"/>
+    <child link="base_footprint"/>
+    <origin xyz="0.0 0.0 -0.15" rpy="0 0 0"/>
     </joint>
     <!-- Base link -->

File: limo_description/urdf/limo_four_diff.xacro (robot description, xacro)
@@ -15,10 +15,10 @@
     <xacro:property name="wheel_length" value="0.0437" />
     <xacro:property name="wheel_radius" value="0.048" />
-  <link name="base_footprint"/>
-  <joint name="base_joint" type="fixed">
-    <parent link="base_footprint"/>
-    <child link="base_link"/>
-    <origin xyz="0.0 0.0 0.15" rpy="0 0 0"/>
-  </joint>
+    <link name="base_footprint"/>
+    <joint name="base_joint" type="fixed">
+    <parent link="base_link"/>
+    <child link="base_footprint"/>
+    <origin xyz="0.0 0.0 -0.15" rpy="0 0 0"/>
+    </joint>
     <!-- Base link -->
     <link name="base_link">

Commit message: started cleaning up navigation

File: limo_description/urdf/limo_ackerman.xacro (robot description, xacro)
@@ -37,6 +37,4 @@
             </geometry>
         </collision>
-    </link>
-    <link name="inertial_link">
         <inertial>
             <origin xyz="0.0 0.0 0.0" />
@@ -47,9 +45,4 @@
         </inertial>
     </link>
-    <joint name="inertial_joint" type="fixed">
-        <origin xyz="0 0 0" rpy="0 0 0" />
-        <parent link="base_link" />
-        <child link="inertial_link" />
-    </joint>
     <xacro:limo_laser parent_prefix="base_link" frame_prefix="laser">
         <origin xyz="0.103 0 -0.034" rpy="0 0 0"/>
@@ -67,53 +60,9 @@
         <origin xyz="${wheelbase/2} ${-track/2} ${wheel_vertical_offset}" rpy="${M_PI} 0 0" />
     </xacro:limo_right_steering_hinge>
-    <link name="rear_left_wheel_link">
-        <inertial>
-            <origin xyz="0 0 0" />
-            <mass value="0.5" />
-            <inertia ixx="0.01055" ixy="0" ixz="0" iyy="0.00075" iyz="0" izz="0.01055" />
-        </inertial>
-        <visual>
-            <origin xyz="0 0 0" rpy="0 0 0" />
-            <geometry>
-                <mesh filename="package://limo_description/meshes/limo_wheel.dae" />
-            </geometry>
-        </visual>
-        <collision>
-            <origin xyz="0 ${wheel_length/2} 0" rpy="1.57 0 0" />
-          <geometry>
-              <cylinder length="${wheel_length}" radius="${wheel_radius}" />
-          </geometry>
-        </collision>
-    </link>
-    <joint name="rear_left_wheel" type="continuous">
-        <parent link="base_link"/>
-        <child link="rear_left_wheel_link"/>
+    <xacro:limo_wheel parent_prefix="base_link" wheel_prefix="rear_left" reflect="1">
         <origin xyz="${-wheelbase/2} ${track/2} ${wheel_vertical_offset}" rpy="0 0 0" />
-        <axis xyz="0 1 0"/>
-    </joint>
-    <link name="rear_right_wheel_link">
-        <inertial>
-            <origin xyz="0 0 0" />
-            <mass value="0.5" />
-            <inertia ixx="0.01055" ixy="0" ixz="0" iyy="0.00075" iyz="0" izz="0.01055" />
-        </inertial>
-        <visual>
-            <origin xyz="0 0 0" rpy="0 0 0" />
-            <geometry>
-                <mesh filename="package://limo_description/meshes/limo_wheel.dae" />
-            </geometry>
-        </visual>
-            <collision>
-                <origin xyz="0 ${wheel_length/2} 0" rpy="1.57 0 0" />
-              <geometry>
-                  <cylinder length="${wheel_length}" radius="${wheel_radius}" />
-              </geometry>
-            </collision>
-        </link>
-        <joint name="rear_right_wheel" type="continuous">
-            <parent link="base_link"/>
-            <child link="rear_right_wheel_link"/>
-            <origin xyz="${-wheelbase/2} ${-track/2} ${wheel_vertical_offset}" rpy="${M_PI} 0 0" />
-            <axis xyz="0 -1 0"/>
-        </joint>
+    </xacro:limo_wheel>
+    <xacro:limo_wheel parent_prefix="base_link" wheel_prefix="rear_right" reflect="-1">
+        <origin xyz="${-wheelbase/2} ${-track/2} ${wheel_vertical_offset}" rpy="${M_PI} 0 0" />
+    </xacro:limo_wheel>
 </robot>

File: limo_description/urdf/limo_four_diff.xacro (robot description, xacro)
@@ -35,6 +35,4 @@
             </geometry>
         </collision>
-    </link>
-    <link name="inertial_link">
         <inertial>
             <origin xyz="0.0 0.0 0.0" />
@@ -45,9 +43,4 @@
         </inertial>
     </link>
-    <joint name="inertial_joint" type="fixed">
-        <origin xyz="0 0 0" rpy="0 0 0" />
-        <parent link="base_link" />
-        <child link="inertial_link" />
-    </joint>
     <xacro:limo_laser parent_prefix="base_link" frame_prefix="laser">
         <origin xyz="0.103 0 -0.034" rpy="0 0 0"/>

File: limo_description/urdf/limo_xacro.xacro (robot description, xacro)
@@ -115,34 +115,5 @@
     </xacro:macro>
     <xacro:macro name="limo_imu" params="parent_prefix frame_prefix  *joint_pose">
-        <link name='${frame_prefix}_link'>
-            <pose>0 0 0 0 0 0</pose>
-            <inertial>
-                <mass value="0.01"/>
-                <origin xyz="0.0 0 0" rpy="0 0 0"/>
-                <inertia
-                    ixx="1e-7" ixy="0" ixz="0"
-                    iyy="1e-7" iyz="0"
-                    izz="1e-7"
-                />
-            </inertial>
-            <visual name='imu_visual'>
-                <origin xyz="0 0 0" rpy="0 0 0"/>
-                <geometry>
-                    <box size="0.001 0.001 0.001"/>
-                </geometry>
-                <material name='imu_material'>
-                    <ambient>0.1 0.1 0.1 1</ambient>
-                    <diffuse>0.1 0.1 0.2 1</diffuse>
-                    <specular>0 0 0 0</specular>
-                    <emissive>0 0 0 1</emissive>
-                </material>
-            </visual>
-            <collision name='imu_collision'>
-                <origin xyz="0 0 0" rpy="0 0 0"/>
-                <geometry>
-                    <box size="0.001 0.001 0.001"/>
-                </geometry>
-            </collision>
-        </link>
+        <link name='${frame_prefix}_link'/>
         <joint type="fixed" name="imu_joint">
             <xacro:insert_block name="joint_pose"/>
@@ -150,7 +121,4 @@
             <parent link="${parent_prefix}"/>
         </joint>
-        <gazebo reference="${frame_prefix}_link">
-            <material>Gazebo/Yellow</material>
-        </gazebo>
     </xacro:macro>
 </robot>

Commit message: So many updated.  Tracker could still use some work.  Ackerman has issues in sim still somehow

File: limo_description/urdf/limo_ackerman.xacro (robot description, xacro)
@@ -7,14 +7,10 @@
     <!-- Variables -->
     <xacro:property name="M_PI" value="3.14159"/>
-    <!-- Vehicle Geometries -->
-    <xacro:property name="base_x_size" value="0.13" />
-    <xacro:property name="base_y_size" value="0.12" />
-    <xacro:property name="base_z_size" value="0.10" />
     <xacro:property name="wheelbase" value="0.2"/>
     <xacro:property name="track" value="0.14"/>
     <xacro:property name="wheel_vertical_offset" value="-0.100998" />
     <xacro:property name="base_mass" value="2.1557"/>
-    <xacro:property name="wheel_length" value="0.045" />
-    <xacro:property name="wheel_radius" value="0.045" />
+    <xacro:property name="wheel_length" value="0.0437" />
+    <xacro:property name="wheel_radius" value="0.048" />
     <link name="base_footprint"/>
     <joint name="base_joint" type="fixed">
@@ -40,7 +36,7 @@
             <origin xyz="0.0 0.0 0.0" />
             <mass value="${base_mass}" />
-            <inertia ixx="0.24" ixy="0" ixz="0"
-                     iyy="0.96" iyz="0"
-                     izz="0.96" />
+            <inertia ixx="0.019264" ixy="0" ixz="0"
+                     iyy="0.029586" iyz="0"
+                     izz="0.02693" />
         </inertial>
     </link>

File: limo_description/urdf/limo_four_diff.xacro (robot description, xacro)
@@ -5,8 +5,4 @@
     <!-- Variables -->
     <xacro:property name="M_PI" value="3.14159"/>
-    <!-- Vehicle Geometries -->
-    <xacro:property name="base_x_size" value="0.13" />
-    <xacro:property name="base_y_size" value="0.12" />
-    <xacro:property name="base_z_size" value="0.1" />
     <xacro:property name="wheelbase" value="0.2"/>
     <xacro:property name="track" value="0.13"/>
@@ -17,7 +13,7 @@
     <link name="base_footprint"/>
     <joint name="base_joint" type="fixed">
-    <parent link="base_link"/>
-    <child link="base_footprint"/>
-    <origin xyz="0.0 0.0 -0.15" rpy="0 0 0"/>
+        <parent link="base_link"/>
+        <child link="base_footprint"/>
+        <origin xyz="0.0 0.0 -0.15" rpy="0 0 0"/>
     </joint>
     <!-- Base link -->
@@ -38,7 +34,7 @@
             <origin xyz="0.0 0.0 0.0" />
             <mass value="${base_mass}" />
-            <inertia ixx="0.24" ixy="0" ixz="0"
-                     iyy="0.96" iyz="0"
-                     izz="0.96" />
+            <inertia ixx="0.019264" ixy="0" ixz="0"
+                     iyy="0.029586" iyz="0"
+                     izz="0.02693" />
         </inertial>
     </link>

File: limo_description/urdf/limo_steering_hinge.xacro (robot description, xacro)
@@ -4,20 +4,12 @@
         <link name="${wheel_prefix}">
             <inertial>
-              <mass value="0.25" />
-              <inertia ixx="0.00525" ixy="0" ixz="0" iyy="0.00035" iyz="0" izz="0.00525" />
-              <origin xyz="0 0 0" />
+                <mass value="0.1"/>
+                <origin xyz="0.0 0 0" rpy="0 0 0"/>
+                <inertia
+                    ixx="1e-6" ixy="0" ixz="0"
+                    iyy="1e-6" iyz="0"
+                    izz="1e-6"
+                />
             </inertial>
-            <visual>
-                <origin xyz="0 0 0" rpy="0 0 0" />
-                <geometry>
-                  <cylinder length="0.0001" radius="0.0001" />
-                </geometry>
-            </visual>
-            <collision>
-              <origin xyz="0 ${wheel_length/2} 0" rpy="1.57 0 0" />
-              <geometry>
-                  <cylinder length="${wheel_length}" radius="${wheel_radius-0.01}" />
-              </geometry>
-            </collision>
         </link>
         <joint name="${wheel_prefix}_wheel" type="revolute">
@@ -31,7 +23,7 @@
         <link name="front_left_wheel_link">
           <inertial>
-            <mass value="0.25" />
-            <inertia ixx="0.00525" ixy="0" ixz="0" iyy="0.00035" iyz="0" izz="0.00525" />
-            <origin xyz="0 0 0" />
+              <origin xyz="0 0.022 0" />
+              <mass value="1.0" />
+              <inertia ixx="0.000147" ixy="0" ixz="0" iyy="0.00023" iyz="0" izz="0.000147" />
           </inertial>
           <visual>
@@ -57,21 +49,13 @@
     <xacro:macro name="limo_right_steering_hinge" params="parent_prefix wheel_prefix *joint_pose">
         <link name="${wheel_prefix}">
-          <inertial>
-            <mass value="0.25" />
-            <inertia ixx="0.00525" ixy="0" ixz="0" iyy="0.00035" iyz="0" izz="0.00525" />
-            <origin xyz="0 0 0" />
-          </inertial>
-            <visual>
-                <origin xyz="0 0 0" rpy="0 0 0" />
-                <geometry>
-                  <cylinder length="0.0001" radius="0.0001" />
-                </geometry>
-            </visual>
-            <collision>
-              <origin xyz="0 ${wheel_length/2} 0" rpy="1.57 0 0" />
-              <geometry>
-                  <cylinder length="${wheel_length}" radius="${wheel_radius-0.01}" />
-              </geometry>
-            </collision>
+            <inertial>
+                <mass value="0.1"/>
+                <origin xyz="0.0 0 0" rpy="0 0 0"/>
+                <inertia
+                    ixx="1e-6" ixy="0" ixz="0"
+                    iyy="1e-6" iyz="0"
+                    izz="1e-6"
+                />
+            </inertial>
         </link>
         <joint name="${wheel_prefix}_wheel" type="revolute">
@@ -85,7 +69,7 @@
         <link name="front_right_wheel_link">
           <inertial>
-            <mass value="0.25" />
-            <inertia ixx="0.00525" ixy="0" ixz="0" iyy="0.00035" iyz="0" izz="0.00525" />
-            <origin xyz="0 0 0" />
+              <origin xyz="0 0.022 0" />
+              <mass value="1.0" />
+              <inertia ixx="0.000147" ixy="0" ixz="0" iyy="0.00023" iyz="0" izz="0.000147" />
           </inertial>
           <visual>

File: limo_description/urdf/limo_xacro.xacro (robot description, xacro)
@@ -4,7 +4,7 @@
         <link name="${wheel_prefix}_wheel_link">
             <inertial>
-                <origin xyz="0 0 0" />
-                <mass value="0.5" />
-                <inertia ixx="0.01055" ixy="0" ixz="0" iyy="0.00075" iyz="0" izz="0.01055" />
+                <origin xyz="0 0.022 0" />
+                <mass value="0.2" />
+                <inertia ixx="0.000147" ixy="0" ixz="0" iyy="0.00023" iyz="0" izz="0.000147" />
             </inertial>
             <visual>
@@ -29,34 +29,5 @@
     </xacro:macro>
     <xacro:macro name="limo_laser" params="parent_prefix frame_prefix *joint_pose">
-        <link name='${frame_prefix}_link'>
-            <pose>0 0 0 0 0 0</pose>
-            <inertial>
-                <mass value="0.1"/>
-                <origin xyz="0.0 0 0" rpy="0 0 0"/>
-                <inertia
-                    ixx="1e-6" ixy="0" ixz="0"
-                    iyy="1e-6" iyz="0"
-                    izz="1e-6"
-                />
-            </inertial>
-            <visual name='laser_visual'>
-                <origin xyz="0 0 0" rpy="0 0 0"/>
-                <geometry>
-                    <cylinder radius="0.02" length="0.01"/>
-                </geometry>
-                <material name='laser_material'>
-                    <ambient>0.1 0.1 0.1 1</ambient>
-                    <diffuse>0.1 0.1 0.2 1</diffuse>
-                    <specular>0 0 0 0</specular>
-                    <emissive>0 0 0 1</emissive>
-                </material>
-            </visual>
-            <collision name='laser_collision'>
-                <origin xyz="0 0 0" rpy="0 0 0"/>
-                <geometry>
-                    <cylinder radius="0.032" length="0.016"/>
-                </geometry>
-            </collision>
-        </link>
+        <link name='${frame_prefix}_link' />
         <joint type="fixed" name="laser_joint">
             <xacro:insert_block name="joint_pose"/>
@@ -64,39 +35,7 @@
             <parent link="${parent_prefix}"/>
         </joint>
-        <gazebo reference="${frame_prefix}_link">
-            <material>Gazebo/Yellow</material>
-        </gazebo>
     </xacro:macro>
     <xacro:macro name="limo_depth_camera" params="parent_prefix frame_prefix *joint_pose">
-        <link name='${frame_prefix}_link'>
-            <pose>0 0 0 0 0 0</pose>
-            <inertial>
-                <mass value="0.1"/>
-                <origin xyz="0.0 0 0" rpy="0 0 0"/>
-                <inertia
-                    ixx="1e-6" ixy="0" ixz="0"
-                    iyy="1e-6" iyz="0"
-                    izz="1e-6"
-                />
-            </inertial>
-            <visual name='depth_camera_visual'>
-                <origin xyz="0 0 0" rpy="0 0 0"/>
-                <geometry>
-                    <box size="0.02 0.06 0.015"/>
-                </geometry>
-                <material name='depth_camera_material'>
-                    <ambient>0.1 0.1 0.1 1</ambient>
-                    <diffuse>0.1 0.1 0.2 1</diffuse>
-                    <specular>0 0 0 0</specular>
-                    <emissive>0 0 0 1</emissive>
-                </material>
-            </visual>
-            <collision name='depth_camera_collision'>
-                <origin xyz="0 0 0" rpy="0 0 0"/>
-                <geometry>
-                    <box size="0.02 0.06 0.015"/>
-                </geometry>
-            </collision>
-        </link>
+        <link name='${frame_prefix}_link' />
         <joint type="fixed" name="depth_camera_joint">
             <xacro:insert_block name="joint_pose"/>
@@ -104,5 +43,5 @@
             <parent link="${parent_prefix}"/>
         </joint>
-        <link name="depth_link"></link>
+        <link name="depth_link" />
         <joint name="${frame_prefix}_to_camera_joint" type="fixed">
             <origin xyz="0 0 0" rpy="${-M_PI/2} 0 ${-M_PI/2} "/>
@@ -110,7 +49,4 @@
             <child link="depth_link"/>
           </joint>
-        <gazebo reference="${frame_prefix}_link">
-            <material>Gazebo/Yellow</material>
-        </gazebo>
     </xacro:macro>
     <xacro:macro name="limo_imu" params="parent_prefix frame_prefix  *joint_pose">
