Commit message: Fixed hinge inertia

File: limo_description/urdf/limo_steering_hinge.xacro (robot description, xacro)
@@ -4,11 +4,7 @@
         <link name="${wheel_prefix}">
             <inertial>
-                <mass value="0.1"/>
-                <origin xyz="0.0 0 0" rpy="0 0 0"/>
-                <inertia
-                    ixx="1e-6" ixy="0" ixz="0"
-                    iyy="1e-6" iyz="0"
-                    izz="1e-6"
-                />
+                <mass value="0.25" />
+                <inertia ixx="0.00525" ixy="0" ixz="0" iyy="0.00035" iyz="0" izz="0.00525" />
+                <origin xyz="0 0 0" />
             </inertial>
         </link>
@@ -50,11 +46,7 @@
         <link name="${wheel_prefix}">
             <inertial>
-                <mass value="0.1"/>
-                <origin xyz="0.0 0 0" rpy="0 0 0"/>
-                <inertia
-                    ixx="1e-6" ixy="0" ixz="0"
-                    iyy="1e-6" iyz="0"
-                    izz="1e-6"
-                />
+                <mass value="0.25" />
+                <inertia ixx="0.00525" ixy="0" ixz="0" iyy="0.00035" iyz="0" izz="0.00525" />
+                <origin xyz="0 0 0" />
             </inertial>
         </link>
